File: tv_b_gone_extended_schematic.brd (EAGLE design)
At the start: 150 x 70 mm, 20 parts, among them IC1 ATMEGA644PV-10PU, IC2 MCP1825S-3302E_DB, J2 2468, J3 2468, Q5 MPS2907A, T1 2N3904, T2 2N3904, T3 2N3904, T4 2N3904, U1 PEC11R-4015F-S0024

Commit message: made progress
Parts:
- added R1, R2: (no value), resistor:0204/5
Connections:
- new net N$10: IC1.5
- new net N$11: IC1.14
- new net N$12: IC1.15
- new net N$13: IC1.16
- new net N$14: IC1.17
- new net N$15: IC1.18
- new net N$16: IC1.19
- new net N$17: IC1.20
- new net N$18: IC1.32
- new net N$19: IC1.21
- new net N$20: R1.1, U1.4
- new net N$7: Q5.B, R2.2
- new net PB0: IC1.1, U1.1
- new net PB1: IC1.2, U1.2
- new net PB2: IC1.3, U1.5
- new net PB3: IC1.4, R2.1
- new net VOUT_REG: IC1.10, IC1.30, IC2.3, PORTA.9, PORTC.9, R1.2
- net GND: now also IC1.11, IC1.31, U1.3
- net VCC: no longer PORTA.9, PORTC.9
Changed lines of the file:
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@@
 <?xml version="1.0" encoding="utf-8"?>
 <!DOCTYPE eagle SYSTEM "eagle.dtd">
-<eagle version="8.5.0">
+<eagle version="8.6.0">
 <drawing>
 <settings>
@@
 <attribute name="SUPPLIER_NAME" value="RS" x="-10" y="-380" size="1" layer="27" display="off"/>
 </element>
+<element name="R1" library="resistor" library_urn="urn:adsk.eagle:library:348" package="0204/5" package3d_urn="urn:adsk.eagle:package:25955/1" value="" x="-30" y="-420"/>
+<element name="R2" library="resistor" library_urn="urn:adsk.eagle:library:348" package="0204/5" package3d_urn="urn:adsk.eagle:package:25955/1" value="" x="-30" y="-440"/>
 </elements>
 <signals>
@@
 <contactref element="J3" pad="2"/>
 <contactref element="J2" pad="2"/>
+<contactref element="U1" pad="3"/>
+<contactref element="IC1" pad="11"/>
+<contactref element="IC1" pad="31"/>
 <wire x1="-19.05" y1="-189.23" x2="-19.05" y2="-205.74" width="0" layer="19" extent="1-1"/>
 <wire x1="-15.24" y1="-151.13" x2="-19.05" y2="-189.23" width="0" layer="19" extent="1-1"/>
@@
 <wire x1="14.13" y1="39.06" x2="14.37" y2="29.06" width="0" layer="19" extent="1-1"/>
 <wire x1="13.89" y1="48.73" x2="14.13" y2="39.06" width="0" layer="19" extent="1-1"/>
-<wire x1="72.95" y1="36.55" x2="14.13" y2="39.06" width="0" layer="19" extent="1-1"/>
+<wire x1="26.3" y1="35.39" x2="14.13" y2="39.06" width="0" layer="19" extent="1-1"/>
+<wire x1="41.54" y1="37.93" x2="26.3" y2="35.39" width="0" layer="19" extent="1-1"/>
+<wire x1="72.95" y1="36.55" x2="41.54" y2="37.93" width="0" layer="19" extent="1-1"/>
 <wire x1="73" y1="45.95" x2="72.95" y2="36.55" width="0" layer="19" extent="1-1"/>
 <wire x1="73" y1="52.05" x2="73" y2="45.95" width="0" layer="19" extent="1-1"/>
 <wire x1="77.57" y1="61.75" x2="73" y2="52.05" width="0" layer="19" extent="1-1"/>
 <wire x1="77.57" y1="12.97" x2="72.95" y2="36.55" width="0" layer="19" extent="1-1"/>
+<wire x1="117.5" y1="10" x2="77.57" y2="12.97" width="0" layer="19" extent="1-1"/>
 <wire x1="127.65" y1="60.625" x2="77.57" y2="61.75" width="0" layer="19" extent="1-1"/>
 </signal>
@@
 <contactref element="C2" pad="+"/>
 <contactref element="ICSP" pad="2"/>
-<contactref element="PORTC" pad="9"/>
-<contactref element="PORTA" pad="9"/>
-<wire x1="77.57" y1="59.21" x2="77.57" y2="10.43" width="0" layer="19" extent="1-1"/>
-<wire x1="-21.59" y1="-205.74" x2="77.57" y2="59.21" width="0" layer="19" extent="1-1"/>
 <wire x1="-21.59" y1="-189.23" x2="-21.59" y2="-205.74" width="0" layer="19" extent="1-1"/>
 <wire x1="-20.32" y1="-151.13" x2="-21.59" y2="-189.23" width="0" layer="19" extent="1-1"/>
-<wire x1="5.35" y1="8.06" x2="-20.32" y2="-151.13" width="0" layer="19" extent="1-1"/>
+<wire x1="-22.86" y1="-68.58" x2="-20.32" y2="-151.13" width="0" layer="19" extent="1-1"/>
+<wire x1="5.35" y1="8.06" x2="-22.86" y2="-68.58" width="0" layer="19" extent="1-1"/>
+<wire x1="5.35" y1="8.06" x2="5.35" y2="8.06" width="0" layer="19" extent="1-16"/>
 <wire x1="5.35" y1="29.06" x2="5.35" y2="8.06" width="0" layer="19" extent="1-1"/>
+<wire x1="5.35" y1="29.06" x2="5.35" y2="29.06" width="0" layer="19" extent="1-16"/>
 <wire x1="5.35" y1="39.06" x2="5.35" y2="29.06" width="0" layer="19" extent="1-1"/>
+<wire x1="5.35" y1="39.06" x2="5.35" y2="39.06" width="0" layer="19" extent="1-16"/>
 <wire x1="5.35" y1="59.06" x2="5.35" y2="39.06" width="0" layer="19" extent="1-1"/>
-<wire x1="-22.86" y1="-68.58" x2="5.35" y2="59.06" width="0" layer="19" extent="1-1"/>
+<wire x1="5.35" y1="59.06" x2="5.35" y2="59.06" width="0" layer="19" extent="1-16"/>
 </signal>
 <signal name="Q5_E">
@@
 <contactref element="J2" pad="1"/>
 </signal>
+<signal name="PB0">
+<contactref element="U1" pad="1"/>
+<contactref element="IC1" pad="1"/>
+<wire x1="41.54" y1="12.53" x2="117.5" y2="7.5" width="0" layer="19" extent="1-1"/>
+</signal>
+<signal name="PB1">
+<contactref element="U1" pad="2"/>
+<contactref element="IC1" pad="2"/>
+<wire x1="41.54" y1="15.07" x2="117.5" y2="12.5" width="0" layer="19" extent="1-1"/>
+</signal>
+<signal name="VOUT_REG">
+<contactref element="IC2" pad="3"/>
+<contactref element="IC1" pad="10"/>
+<contactref element="PORTA" pad="9"/>
+<contactref element="PORTC" pad="9"/>
+<contactref element="IC1" pad="30"/>
+<contactref element="R1" pad="2"/>
+<wire x1="77.57" y1="10.43" x2="-27.46" y2="-420" width="0" layer="19" extent="1-1"/>
+<wire x1="75.3" y1="45.95" x2="77.57" y2="10.43" width="0" layer="19" extent="1-1"/>
+<wire x1="77.57" y1="59.21" x2="75.3" y2="45.95" width="0" layer="19" extent="1-1"/>
+<wire x1="41.54" y1="35.39" x2="75.3" y2="45.95" width="0" layer="19" extent="1-1"/>
+<wire x1="26.3" y1="37.93" x2="41.54" y2="35.39" width="0" layer="19" extent="1-1"/>
+</signal>
+<signal name="N$10">
+<contactref element="IC1" pad="5"/>
+</signal>
+<signal name="N$11">
+<contactref element="IC1" pad="14"/>
+</signal>
+<signal name="N$12">
+<contactref element="IC1" pad="15"/>
+</signal>
+<signal name="N$13">
+<contactref element="IC1" pad="16"/>
+</signal>
+<signal name="N$14">
+<contactref element="IC1" pad="17"/>
+</signal>
+<signal name="N$15">
+<contactref element="IC1" pad="18"/>
+</signal>
+<signal name="N$16">
+<contactref element="IC1" pad="19"/>
+</signal>
+<signal name="N$17">
+<contactref element="IC1" pad="20"/>
+</signal>
+<signal name="N$18">
+<contactref element="IC1" pad="32"/>
+</signal>
+<signal name="N$19">
+<contactref element="IC1" pad="21"/>
+</signal>
+<signal name="N$20">
+<contactref element="U1" pad="4"/>
+<contactref element="R1" pad="1"/>
+<wire x1="103" y1="7.5" x2="-32.54" y2="-420" width="0" layer="19" extent="1-1"/>
+</signal>
+<signal name="PB2">
+<contactref element="U1" pad="5"/>
+<contactref element="IC1" pad="3"/>
+<wire x1="41.54" y1="17.61" x2="103" y2="12.5" width="0" layer="19" extent="1-1"/>
+</signal>
+<signal name="N$7">
+<contactref element="Q5" pad="B"/>
+<contactref element="R2" pad="2"/>
+<wire x1="-20.32" y1="-68.58" x2="-27.46" y2="-440" width="0" layer="19" extent="1-1"/>
+</signal>
+<signal name="PB3">
+<contactref element="R2" pad="1"/>
+<contactref element="IC1" pad="4"/>
+<wire x1="41.54" y1="20.15" x2="-32.54" y2="-440" width="0" layer="19" extent="1-1"/>
+</signal>
 </signals>

Commit message: made progress
Parts:
- moved R1 459.5 mm to (72.0, 28.0)
Connections:
- removed net N$20: R1.1, U1.4
- net GND: now also U1.5
- net PB2: now also R1.1, U1.4; no longer U1.5
- net VCC: no longer LED1.A, LED1.A2, LED2.A, LED2.A2, LED3.A, LED3.A2, LED4.A, LED4.A2
- net VOUT_REG: now also LED1.A, LED1.A2, LED2.A, LED2.A2, LED3.A, LED3.A2, LED4.A, LED4.A2
Changed lines of the file:
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@@
 <setting verticaltext="up"/>
 </settings>
-<grid distance="10" unitdist="mm" unit="mm" style="lines" multiple="1" display="yes" altdistance="1" altunitdist="mm" altunit="mm"/>
+<grid distance="10" unitdist="mm" unit="mm" style="lines" multiple="1" display="no" altdistance="1" altunitdist="mm" altunit="mm"/>
 <layers>
 <layer number="1" name="Top" color="4" fill="1" visible="yes" active="yes"/>
@@
 <attribute name="SUPPLIER_NAME" value="RS" x="-10" y="-380" size="1" layer="27" display="off"/>
 </element>
-<element name="R1" library="resistor" library_urn="urn:adsk.eagle:library:348" package="0204/5" package3d_urn="urn:adsk.eagle:package:25955/1" value="" x="-30" y="-420"/>
+<element name="R1" library="resistor" library_urn="urn:adsk.eagle:library:348" package="0204/5" package3d_urn="urn:adsk.eagle:package:25955/1" value="" x="72" y="28"/>
 <element name="R2" library="resistor" library_urn="urn:adsk.eagle:library:348" package="0204/5" package3d_urn="urn:adsk.eagle:package:25955/1" value="" x="-30" y="-440"/>
 </elements>
@@
 <contactref element="IC1" pad="11"/>
 <contactref element="IC1" pad="31"/>
+<contactref element="U1" pad="5"/>
 <wire x1="-19.05" y1="-189.23" x2="-19.05" y2="-205.74" width="0" layer="19" extent="1-1"/>
 <wire x1="-15.24" y1="-151.13" x2="-19.05" y2="-189.23" width="0" layer="19" extent="1-1"/>
@@
 <wire x1="77.57" y1="61.75" x2="73" y2="52.05" width="0" layer="19" extent="1-1"/>
 <wire x1="77.57" y1="12.97" x2="72.95" y2="36.55" width="0" layer="19" extent="1-1"/>
-<wire x1="117.5" y1="10" x2="77.57" y2="12.97" width="0" layer="19" extent="1-1"/>
+<wire x1="103" y1="12.5" x2="77.57" y2="12.97" width="0" layer="19" extent="1-1"/>
+<wire x1="117.5" y1="10" x2="103" y2="12.5" width="0" layer="19" extent="1-1"/>
 <wire x1="127.65" y1="60.625" x2="77.57" y2="61.75" width="0" layer="19" extent="1-1"/>
 </signal>
 <signal name="VCC">
 <contactref element="Q5" pad="E"/>
-<contactref element="LED3" pad="A"/>
-<contactref element="LED3" pad="A2"/>
-<contactref element="LED1" pad="A"/>
-<contactref element="LED1" pad="A2"/>
-<contactref element="LED2" pad="A"/>
-<contactref element="LED2" pad="A2"/>
-<contactref element="LED4" pad="A"/>
-<contactref element="LED4" pad="A2"/>
 <contactref element="C1" pad="1"/>
 <contactref element="C2" pad="+"/>
@@
 <wire x1="-20.32" y1="-151.13" x2="-21.59" y2="-189.23" width="0" layer="19" extent="1-1"/>
 <wire x1="-22.86" y1="-68.58" x2="-20.32" y2="-151.13" width="0" layer="19" extent="1-1"/>
-<wire x1="5.35" y1="8.06" x2="-22.86" y2="-68.58" width="0" layer="19" extent="1-1"/>
-<wire x1="5.35" y1="8.06" x2="5.35" y2="8.06" width="0" layer="19" extent="1-16"/>
-<wire x1="5.35" y1="29.06" x2="5.35" y2="8.06" width="0" layer="19" extent="1-1"/>
-<wire x1="5.35" y1="29.06" x2="5.35" y2="29.06" width="0" layer="19" extent="1-16"/>
-<wire x1="5.35" y1="39.06" x2="5.35" y2="29.06" width="0" layer="19" extent="1-1"/>
-<wire x1="5.35" y1="39.06" x2="5.35" y2="39.06" width="0" layer="19" extent="1-16"/>
-<wire x1="5.35" y1="59.06" x2="5.35" y2="39.06" width="0" layer="19" extent="1-1"/>
-<wire x1="5.35" y1="59.06" x2="5.35" y2="59.06" width="0" layer="19" extent="1-16"/>
 </signal>
 <signal name="Q5_E">
@@
 <contactref element="U1" pad="1"/>
 <contactref element="IC1" pad="1"/>
-<wire x1="41.54" y1="12.53" x2="117.5" y2="7.5" width="0" layer="19" extent="1-1"/>
+<wire x1="117.5" y1="7.5" x2="41.54" y2="12.53" width="0" layer="19" extent="1-1"/>
 </signal>
 <signal name="PB1">
 <contactref element="U1" pad="2"/>
 <contactref element="IC1" pad="2"/>
-<wire x1="41.54" y1="15.07" x2="117.5" y2="12.5" width="0" layer="19" extent="1-1"/>
+<wire x1="117.5" y1="12.5" x2="41.54" y2="15.07" width="0" layer="19" extent="1-1"/>
 </signal>
 <signal name="VOUT_REG">
@@
 <contactref element="IC1" pad="30"/>
 <contactref element="R1" pad="2"/>
-<wire x1="77.57" y1="10.43" x2="-27.46" y2="-420" width="0" layer="19" extent="1-1"/>
-<wire x1="75.3" y1="45.95" x2="77.57" y2="10.43" width="0" layer="19" extent="1-1"/>
+<contactref element="LED3" pad="A"/>
+<contactref element="LED3" pad="A2"/>
+<contactref element="LED1" pad="A"/>
+<contactref element="LED1" pad="A2"/>
+<contactref element="LED2" pad="A"/>
+<contactref element="LED2" pad="A2"/>
+<contactref element="LED4" pad="A"/>
+<contactref element="LED4" pad="A2"/>
+<wire x1="74.54" y1="28" x2="5.35" y2="8.06" width="0" layer="19" extent="1-1"/>
+<wire x1="5.35" y1="8.06" x2="5.35" y2="8.06" width="0" layer="19" extent="1-16"/>
+<wire x1="5.35" y1="29.06" x2="5.35" y2="8.06" width="0" layer="19" extent="1-1"/>
+<wire x1="5.35" y1="29.06" x2="5.35" y2="29.06" width="0" layer="19" extent="1-16"/>
+<wire x1="5.35" y1="39.06" x2="5.35" y2="29.06" width="0" layer="19" extent="1-1"/>
+<wire x1="5.35" y1="39.06" x2="5.35" y2="39.06" width="0" layer="19" extent="1-16"/>
+<wire x1="5.35" y1="59.06" x2="5.35" y2="39.06" width="0" layer="19" extent="1-1"/>
+<wire x1="5.35" y1="59.06" x2="5.35" y2="59.06" width="0" layer="19" extent="1-16"/>
+<wire x1="26.3" y1="37.93" x2="5.35" y2="39.06" width="0" layer="19" extent="1-1"/>
+<wire x1="41.54" y1="35.39" x2="26.3" y2="37.93" width="0" layer="19" extent="1-1"/>
+<wire x1="75.3" y1="45.95" x2="41.54" y2="35.39" width="0" layer="19" extent="1-1"/>
 <wire x1="77.57" y1="59.21" x2="75.3" y2="45.95" width="0" layer="19" extent="1-1"/>
-<wire x1="41.54" y1="35.39" x2="75.3" y2="45.95" width="0" layer="19" extent="1-1"/>
-<wire x1="26.3" y1="37.93" x2="41.54" y2="35.39" width="0" layer="19" extent="1-1"/>
+<wire x1="77.57" y1="10.43" x2="75.3" y2="45.95" width="0" layer="19" extent="1-1"/>
 </signal>
 <signal name="N$10">
@@
 <contactref element="IC1" pad="21"/>
 </signal>
-<signal name="N$20">
+<signal name="PB2">
+<contactref element="IC1" pad="3"/>
 <contactref element="U1" pad="4"/>
 <contactref element="R1" pad="1"/>
-<wire x1="103" y1="7.5" x2="-32.54" y2="-420" width="0" layer="19" extent="1-1"/>
-</signal>
-<signal name="PB2">
-<contactref element="U1" pad="5"/>
-<contactref element="IC1" pad="3"/>
-<wire x1="41.54" y1="17.61" x2="103" y2="12.5" width="0" layer="19" extent="1-1"/>
+<wire x1="69.46" y1="28" x2="41.54" y2="17.61" width="0" layer="19" extent="1-1"/>
+<wire x1="103" y1="7.5" x2="41.54" y2="17.61" width="0" layer="19" extent="1-1"/>
 </signal>
 <signal name="N$7">

Commit message: made progress - Thanks Kier :)
Parts:
- removed J2, J3: 2468, SamacSys_Parts:2468
- added BAT_1, BAT_2: 2468, SamacSys_Parts:2468
- added R3: (no value), rcl:0204/7
- added S1: 1825910-6, SamacSys_Parts:1825910-6
- C1: value 0.1uF -> 100nF
- C2: value 100uF -> 100nF; device rcl-ez:E2,5-5 -> rcl-ez:C025-025X050
- moved R2 486.4 mm to (42.0, 41.0), turned to 90 degrees
- moved C2 248.7 mm to (47.0, 33.6), turned to 180 degrees
- moved ICSP 219.3 mm to (60.2, 52.6)
- moved C1 210.3 mm to (44.5, 10.8), turned to 180 degrees
- moved Q5 85.7 mm to (14.0, 10.0), turned to 270 degrees
- moved PORTA 52.9 mm to (23.5, 40.5), turned to 90 degrees
- moved IC1 46.6 mm to (22.9, 14.3), turned to 270 degrees
- moved XTL1 38.9 mm to (34.0, 35.5), turned to 180 degrees
- moved IC2 33.1 mm to (40.0, 52.0), turned to 180 degrees
- moved PORTC 29.2 mm to (77.5, 40.5), turned to 90 degrees
- moved R1 29.1 mm to (46.0, 41.0), turned to 90 degrees
- moved U1 21.2 mm to (89.0, 13.0)
- moved LED3 12.3 mm to (5.35, 48.0)
- moved LED1 4.00 mm to (5.35, 36.3)
- moved LED2 4.00 mm to (5.35, 26.3)
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Connections:
- removed net N$1: IC2.1
- removed net N$4: J3.1
- removed net N$5: J2.1
- removed net VCC: C1.1, C2.+, ICSP.2, Q5.E
- new net VIN_REG: BAT_1.1, BAT_2.1, IC2.1, LED1.A, LED1.A2, LED2.A, LED2.A2, LED3.A, LED3.A2, LED4.A, LED4.A2
- net GND: now also BAT_1.2, BAT_2.2, C2.2, S1.3, S1.4; no longer C2.-, J2.2, J3.2
- net RESET: now also R3.2, S1.1, S1.2
- net VOUT_REG: now also C1.1, C2.1, ICSP.2, Q5.E, R3.1; no longer LED1.A, LED1.A2, LED2.A, LED2.A2, LED3.A, LED3.A2, LED4.A, LED4.A2
Routing:
- net GND: track 0.00 -> 15.5 mm
- net XTAL1: track 0.00 -> 12.6 mm
- net XTAL2: track 0.00 -> 10.3 mm
- net N$8: track 0.00 -> 9.89 mm
- net N$3: track 0.00 -> 9.27 mm
- net N$6: track 0.00 -> 9.03 mm
- net N$2: track 0.00 -> 8.95 mm, vias 0 -> 1
Other:
- board size 150 x 70 mm -> 101 x 58 mm

Commit message: routing
Parts:
- moved C1 2.54 mm to (47.0, 10.8), turned to 0 degrees
- flipped IC2 to the bottom
Connections:
- net N$2 renamed T1_C
- net N$3 renamed T2_C
- net N$6 renamed T3_C
- net N$8 renamed T4_C
Routing:
- net GND: track 15.5 -> 310.4 mm, vias 0 -> 6
- net VOUT_REG: track 0.00 -> 159.5 mm, vias 0 -> 6
- net VIN_REG: track 0.00 -> 116.3 mm, vias 0 -> 5
- net Q5_E: track 0.00 -> 114.2 mm, vias 0 -> 1
- net PA1: track 0.00 -> 91.5 mm, vias 0 -> 7
- net PC0: track 0.00 -> 84.7 mm, vias 0 -> 1
- net PC1: track 0.00 -> 79.1 mm
- net PC2: track 0.00 -> 77.9 mm, vias 0 -> 1
- net PA0: track 0.00 -> 73.8 mm, vias 0 -> 4
- net PC4: track 0.00 -> 71.3 mm
- net PC3: track 0.00 -> 69.6 mm, vias 0 -> 1
- net PC6: track 0.00 -> 67.1 mm, vias 0 -> 1
- net PC5: track 0.00 -> 65.3 mm, vias 0 -> 1
- net PB1: track 0.00 -> 64.2 mm, vias 0 -> 1
- net PA2: track 0.00 -> 63.3 mm
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Other:
- board text added: "Anton Nikitin Project Vostok 2018 Version 1"
