File: tv_b_gone_extended_schematic.brd (EAGLE design)
At the start: 101 x 58 mm, 24 parts, among them IC1 ATMEGA644PV-10PU, IC2 MCP1825S-3302E_DB, Q5 MPS2907A, T1 2N3904, T2 2N3904, T3 2N3904, T4 2N3904, U1 PEC11R-4015F-S0024

Commit message: remove garbage files and add detail to schem
Other:
- board text added: "Based upon the TV-B-Gone By Mitch Altman"
- board text removed: "IR LED Circuit taken from TV-B-Gone By Mitch Altman"
Changed lines of the file:
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@@
 Project Vostok
 2018 Version 1</text>
-<text x="0.635" y="59.69" size="0.6096" layer="25">IR LED Circuit taken from TV-B-Gone
+<text x="0.635" y="59.69" size="0.6096" layer="25">Based upon the TV-B-Gone
 By Mitch Altman</text>
 <text x="22.225" y="19.685" size="0.6096" layer="25" rot="R90">ATMega644P</text>
