File: tv_b_gone_extended_schematic.sch (EAGLE design)
At the start: 20 parts, among them IC1 ATMEGA644PV-10PU, IC2 MCP1825S-3302E_DB, J2 2468, J3 2468, Q5 MPS2907A, T1 2N3904, T2 2N3904, T3 2N3904, T4 2N3904, U1 PEC11R-4015F-S0024

Commit message: made progress
Parts:
- added R1, R2: (no value), resistor:R-EU_0204/5
Connections:
- new net N$10: IC1.PB4
- new net N$11: IC1.PD0
- new net N$12: IC1.PD1
- new net N$13: IC1.PD2
- new net N$14: IC1.PD3
- new net N$15: IC1.PD4
- new net N$16: IC1.PD5
- new net N$17: IC1.PD6
- new net N$18: IC1.AREF
- new net N$19: IC1.PD7
- new net N$20: R1.1, U1.1
- new net N$7: Q5.B, R2.2
- new net PB0: IC1.PB0, U1.A
- new net PB1: IC1.PB1, U1.B
- new net PB2: IC1.PB2, U1.2
- new net PB3: IC1.PB3, R2.1
- new net VOUT_REG: IC1.AVCC, IC1.VCC, IC2.VOUT, PORTA.9, PORTC.9, R1.2
- net GND: now also IC1.GND, IC1.GND_2, U1.C
- net VCC: no longer PORTA.9, PORTC.9
Other:
- note added: "PB0"
- note added: "PB1"
- note added: "PB2"
- note added: "PB3"
- note added: "PB4"
- note added: "UNUSED"
- note added: "VOUT_REG"
- moved on the sheet: C1, C2, ICSP, PORTA, PORTC, Q5, U1, XTL1

Commit message: made progress
Connections:
- removed net N$20: R1.1, U1.1
- net GND: now also U1.2
- net PB2: now also R1.1, U1.1; no longer U1.2
- net VCC: no longer LED1.A, LED1.A1, LED2.A, LED2.A1, LED3.A, LED3.A1, LED4.A, LED4.A1
- net VOUT_REG: now also LED1.A, LED1.A1, LED2.A, LED2.A1, LED3.A, LED3.A1, LED4.A, LED4.A1
Changed lines of the file:
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@@
 <part name="LED2" library="tvbgone" deviceset="LED" device=""/>
 <part name="LED4" library="tvbgone" deviceset="LED" device=""/>
-<part name="P+2" library="supply1" library_urn="urn:adsk.eagle:library:371" deviceset="VCC" device=""/>
-<part name="P+3" library="supply1" library_urn="urn:adsk.eagle:library:371" deviceset="VCC" device=""/>
-<part name="P+4" library="supply1" library_urn="urn:adsk.eagle:library:371" deviceset="VCC" device=""/>
-<part name="P+5" library="supply1" library_urn="urn:adsk.eagle:library:371" deviceset="VCC" device=""/>
 <part name="ICSP" library="adaprog" deviceset="PINHD-2X3" device="THM"/>
 <part name="XTL1" library="digg" deviceset="CERMOSCILL" device="" value="8.0MHz"/>
@@
 <part name="R1" library="resistor" library_urn="urn:adsk.eagle:library:348" deviceset="R-EU_" device="0204/5" package3d_urn="urn:adsk.eagle:package:25955/1"/>
 <part name="R2" library="resistor" library_urn="urn:adsk.eagle:library:348" deviceset="R-EU_" device="0204/5" package3d_urn="urn:adsk.eagle:package:25955/1"/>
+<part name="GND14" library="supply1" library_urn="urn:adsk.eagle:library:371" deviceset="GND" device=""/>
 </parts>
 <sheets>
@@
 <text x="180.34" y="35.56" size="1.778" layer="95">UNUSED</text>
 <text x="198.12" y="27.94" size="1.778" layer="95">VOUT_REG</text>
-<text x="198.12" y="10.16" size="1.778" layer="95">PB2</text>
 <text x="48.26" y="30.48" size="1.778" layer="95">PB3</text>
+<text x="58.42" y="83.82" size="1.778" layer="95" rot="R90">VOUT_REG</text>
+<text x="73.66" y="83.82" size="1.778" layer="95" rot="R90">VOUT_REG</text>
+<text x="88.9" y="83.82" size="1.778" layer="95" rot="R90">VOUT_REG</text>
+<text x="104.14" y="83.82" size="1.778" layer="95" rot="R90">VOUT_REG</text>
+<text x="203.2" y="12.7" size="1.778" layer="95">PB2</text>
 </plain>
 <instances>
@@
 <instance part="LED2" gate="G$1" x="88.9" y="73.66"/>
 <instance part="LED4" gate="G$1" x="104.14" y="73.66"/>
-<instance part="P+2" gate="VCC" x="58.42" y="86.36"/>
-<instance part="P+3" gate="VCC" x="73.66" y="86.36"/>
-<instance part="P+4" gate="VCC" x="88.9" y="86.36"/>
-<instance part="P+5" gate="VCC" x="104.14" y="86.36"/>
 <instance part="ICSP" gate="G$1" x="259.08" y="-2.54"/>
 <instance part="XTL1" gate="G$1" x="264.16" y="-35.56" smashed="yes" rot="R270">
@@
 <instance part="R1" gate="G$1" x="198.12" y="20.32" rot="R90"/>
 <instance part="R2" gate="G$1" x="63.5" y="30.48"/>
+<instance part="GND14" gate="1" x="203.2" y="2.54"/>
 </instances>
 <busses>
@@
 <pinref part="GND13" gate="1" pin="GND"/>
 </segment>
+<segment>
+<pinref part="U1" gate="G$1" pin="2"/>
+<wire x1="195.58" y1="10.16" x2="203.2" y2="10.16" width="0.1524" layer="91"/>
+<wire x1="203.2" y1="10.16" x2="203.2" y2="5.08" width="0.1524" layer="91"/>
+<pinref part="GND14" gate="1" pin="GND"/>
+</segment>
 </net>
 <net name="VCC" class="0">
@@
 <wire x1="81.28" y1="35.56" x2="81.28" y2="40.64" width="0.1524" layer="91"/>
 <pinref part="P+1" gate="VCC" pin="VCC"/>
-</segment>
-<segment>
-<pinref part="LED3" gate="G$1" pin="A"/>
-<pinref part="LED3" gate="G$1" pin="A1"/>
-<wire x1="58.42" y1="78.74" x2="60.96" y2="78.74" width="0.1524" layer="91"/>
-<wire x1="58.42" y1="78.74" x2="58.42" y2="83.82" width="0.1524" layer="91"/>
-<junction x="58.42" y="78.74"/>
-<pinref part="P+2" gate="VCC" pin="VCC"/>
-</segment>
-<segment>
-<pinref part="LED1" gate="G$1" pin="A"/>
-<pinref part="LED1" gate="G$1" pin="A1"/>
-<wire x1="73.66" y1="78.74" x2="76.2" y2="78.74" width="0.1524" layer="91"/>
-<wire x1="73.66" y1="78.74" x2="73.66" y2="83.82" width="0.1524" layer="91"/>
-<junction x="73.66" y="78.74"/>
-<pinref part="P+3" gate="VCC" pin="VCC"/>
-</segment>
-<segment>
-<pinref part="LED2" gate="G$1" pin="A"/>
-<pinref part="LED2" gate="G$1" pin="A1"/>
-<wire x1="88.9" y1="78.74" x2="91.44" y2="78.74" width="0.1524" layer="91"/>
-<wire x1="88.9" y1="78.74" x2="88.9" y2="83.82" width="0.1524" layer="91"/>
-<junction x="88.9" y="78.74"/>
-<pinref part="P+4" gate="VCC" pin="VCC"/>
-</segment>
-<segment>
-<pinref part="LED4" gate="G$1" pin="A"/>
-<pinref part="LED4" gate="G$1" pin="A1"/>
-<wire x1="104.14" y1="78.74" x2="106.68" y2="78.74" width="0.1524" layer="91"/>
-<wire x1="104.14" y1="78.74" x2="104.14" y2="83.82" width="0.1524" layer="91"/>
-<junction x="104.14" y="78.74"/>
-<pinref part="P+5" gate="VCC" pin="VCC"/>
 </segment>
 <segment>
@@
 <wire x1="198.12" y1="25.4" x2="198.12" y2="27.94" width="0.1524" layer="91"/>
 </segment>
+<segment>
+<pinref part="LED3" gate="G$1" pin="A"/>
+<pinref part="LED3" gate="G$1" pin="A1"/>
+<wire x1="58.42" y1="78.74" x2="60.96" y2="78.74" width="0.1524" layer="91"/>
+<wire x1="58.42" y1="78.74" x2="58.42" y2="83.82" width="0.1524" layer="91"/>
+<junction x="58.42" y="78.74"/>
+</segment>
+<segment>
+<pinref part="LED1" gate="G$1" pin="A"/>
+<pinref part="LED1" gate="G$1" pin="A1"/>
+<wire x1="73.66" y1="78.74" x2="76.2" y2="78.74" width="0.1524" layer="91"/>
+<wire x1="73.66" y1="78.74" x2="73.66" y2="83.82" width="0.1524" layer="91"/>
+<junction x="73.66" y="78.74"/>
+</segment>
+<segment>
+<pinref part="LED2" gate="G$1" pin="A"/>
+<pinref part="LED2" gate="G$1" pin="A1"/>
+<wire x1="88.9" y1="78.74" x2="91.44" y2="78.74" width="0.1524" layer="91"/>
+<wire x1="88.9" y1="78.74" x2="88.9" y2="83.82" width="0.1524" layer="91"/>
+<junction x="88.9" y="78.74"/>
+</segment>
+<segment>
+<pinref part="LED4" gate="G$1" pin="A"/>
+<pinref part="LED4" gate="G$1" pin="A1"/>
+<wire x1="104.14" y1="78.74" x2="106.68" y2="78.74" width="0.1524" layer="91"/>
+<wire x1="104.14" y1="78.74" x2="104.14" y2="83.82" width="0.1524" layer="91"/>
+<junction x="104.14" y="78.74"/>
+</segment>
 </net>
 <net name="N$10" class="0">
@@
 </segment>
 </net>
-<net name="N$20" class="0">
+<net name="PB2" class="0">
+<segment>
+<pinref part="IC1" gate="G$1" pin="PB2"/>
+<wire x1="144.78" y1="78.74" x2="134.62" y2="78.74" width="0.1524" layer="91"/>
+</segment>
 <segment>
 <pinref part="U1" gate="G$1" pin="1"/>
@@
 <wire x1="198.12" y1="12.7" x2="198.12" y2="15.24" width="0.1524" layer="91"/>
 <pinref part="R1" gate="G$1" pin="1"/>
-</segment>
-</net>
-<net name="PB2" class="0">
-<segment>
-<pinref part="U1" gate="G$1" pin="2"/>
-<wire x1="195.58" y1="10.16" x2="198.12" y2="10.16" width="0.1524" layer="91"/>
-</segment>
-<segment>
-<pinref part="IC1" gate="G$1" pin="PB2"/>
-<wire x1="144.78" y1="78.74" x2="134.62" y2="78.74" width="0.1524" layer="91"/>
-</segment>
-</net>
+<wire x1="198.12" y1="12.7" x2="203.2" y2="12.7" width="0.1524" layer="91"/>
+<junction x="198.12" y="12.7"/>
+</segment>
+</net>

Commit message: made progress - Thanks Kier :)
Parts:
- removed J2: 2468, SamacSys_Parts:2468
- added BAT_2: 2468, SamacSys_Parts:2468
- added R3: (no value), rcl:R-EU_0204/7
- added S1: 1825910-6, SamacSys_Parts:1825910-6
- C1: value 0.1uF -> 100nF
- C2: value 100uF -> 100nF; device rcl-ez:CPOL-USE2.5-5 -> rcl-ez:C-US025-025X050
- renumbered J3 to BAT_1
Connections:
- removed net N$1: IC2.VIN
- removed net N$4: BAT_1.POS
- removed net N$5: J2.POS
- removed net VCC: C1.1, C2.+, ICSP.2, Q5.E
- new net VIN_REG: BAT_1.POS, BAT_2.POS, IC2.VIN, LED1.A, LED1.A1, LED2.A, LED2.A1, LED3.A, LED3.A1, LED4.A, LED4.A1
- net GND: now also BAT_2.NEG, C2.2, S1.3, S1.4; no longer C2.-, J2.NEG
- net RESET: now also R3.2, S1.1, S1.2
- net VOUT_REG: now also C1.1, C2.1, ICSP.2, Q5.E, R3.1; no longer LED1.A, LED1.A1, LED2.A, LED2.A1, LED3.A, LED3.A1, LED4.A, LED4.A1
Other:
- note removed: "PB4"
- note removed: "Q5_E"
- note removed: "VIN_REG"
- moved on the sheet: C1

Commit message: routing
Connections:
- net N$2 renamed T1_C
- net N$3 renamed T2_C
- net N$6 renamed T3_C
- net N$8 renamed T4_C
Changed lines of the file:
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@@
 <?xml version="1.0" encoding="utf-8"?>
 <!DOCTYPE eagle SYSTEM "eagle.dtd">
-<eagle version="8.5.0">
+<eagle version="8.6.0">
 <drawing>
 <settings>
@@
 </segment>
 </net>
-<net name="N$2" class="0">
+<net name="T1_C" class="0">
 <segment>
 <pinref part="LED3" gate="G$1" pin="C"/>
@@
 </segment>
 </net>
-<net name="N$3" class="0">
+<net name="T2_C" class="0">
 <segment>
 <pinref part="LED1" gate="G$1" pin="C"/>
@@
 </segment>
 </net>
-<net name="N$6" class="0">
+<net name="T3_C" class="0">
 <segment>
 <pinref part="LED2" gate="G$1" pin="C"/>
@@
 </segment>
 </net>
-<net name="N$8" class="0">
+<net name="T4_C" class="0">
 <segment>
 <pinref part="LED4" gate="G$1" pin="C"/>
