File: board files/v1.1/project_vostok_(tv_b_gone_extended)_v1.1.brd (EAGLE design)
At the start: 100 x 80 mm, 25 parts, among them IC1 ATMEGA644PV-10PU, IC2 MCP1825S-3302E_DB, Q5 MPS2907A, T1 2N3904, T2 2N3904, T3 2N3904, T4 2N3904, U1 PEC11R-4015F-S0024

Commit message: modify port
Connections:
- removed net N$1: PORTC.10
- removed net N$2: PORTA.10
- new net N$4: R3.2, S1.2
- net GND: now also PORTA.2, PORTC.2
- net PA0: now also PORTA.10; no longer PORTA.1
- net PA1: now also PORTA.9; no longer PORTA.2
- net PA2: now also PORTA.8; no longer PORTA.3
- net PA3: now also PORTA.7; no longer PORTA.4
- net PA4: now also PORTA.6; no longer PORTA.5
- net PA5: now also PORTA.5; no longer PORTA.6
- net PA6: now also PORTA.4; no longer PORTA.7
- net PA7: now also PORTA.3; no longer PORTA.8
- net PC0: now also PORTC.10; no longer PORTC.1
- net PC1: now also PORTC.9; no longer PORTC.2
- net PC2: now also PORTC.8; no longer PORTC.3
- net PC3: now also PORTC.7; no longer PORTC.4
- net PC4: now also PORTC.6; no longer PORTC.5
- net PC5: now also PORTC.5; no longer PORTC.6
- net PC6: now also PORTC.4; no longer PORTC.7
- net PC7: now also PORTC.3; no longer PORTC.8
- net RESET: no longer R3.2, S1.2
- net VOUT_REG: now also PORTA.1, PORTC.1; no longer PORTA.9, PORTC.9
Changed lines of the file:
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@@
 <contactref element="S1" pad="4"/>
 <contactref element="LED5" pad="A"/>
+<contactref element="PORTC" pad="2"/>
+<contactref element="PORTA" pad="2"/>
 <wire x1="7.11" y1="-173.99" x2="8.89" y2="-229.87" width="0" layer="19" extent="1-1"/>
 <wire x1="13.21" y1="-173.99" x2="7.11" y2="-173.99" width="0" layer="19" extent="1-1"/>
@@
 <wire x1="31.04" y1="-122.21" x2="31.04" y2="-126.71" width="0" layer="19" extent="1-1"/>
 <wire x1="13.97" y1="-123.19" x2="31.04" y2="-122.21" width="0" layer="19" extent="1-1"/>
-<wire x1="97.79" y1="-143.51" x2="31.75" y2="-143.51" width="0" layer="19" extent="1-1"/>
+<wire x1="53.34" y1="-121.92" x2="31.04" y2="-122.21" width="0" layer="19" extent="1-1"/>
+<wire x1="78.74" y1="-121.92" x2="53.34" y2="-121.92" width="0" layer="19" extent="1-1"/>
+<wire x1="97.79" y1="-143.51" x2="78.74" y2="-121.92" width="0" layer="19" extent="1-1"/>
 <wire x1="116.84" y1="-143.51" x2="97.79" y2="-143.51" width="0" layer="19" extent="1-1"/>
 <wire x1="107.95" y1="-123.19" x2="116.84" y2="-143.51" width="0" layer="19" extent="1-1"/>
@@
 <contactref element="ICSP" pad="5"/>
 <contactref element="S1" pad="1"/>
-<contactref element="S1" pad="2"/>
-<contactref element="R3" pad="2"/>
-<wire x1="13.97" y1="-125.73" x2="15.24" y2="-200.66" width="0" layer="19" extent="1-1"/>
-<wire x1="37.54" y1="-126.71" x2="13.97" y2="-125.73" width="0" layer="19" extent="1-1"/>
-<wire x1="37.54" y1="-122.21" x2="37.54" y2="-126.71" width="0" layer="19" extent="1-1"/>
+<wire x1="37.54" y1="-122.21" x2="13.97" y2="-125.73" width="0" layer="19" extent="1-1"/>
 <wire x1="7.62" y1="-27.94" x2="13.97" y2="-125.73" width="0" layer="19" extent="1-1"/>
 </signal>
 <signal name="PA0">
 <contactref element="IC1" pad="40"/>
-<contactref element="PORTA" pad="1"/>
-<wire x1="22.86" y1="-7.62" x2="53.34" y2="-124.46" width="0" layer="19" extent="1-1"/>
+<contactref element="PORTA" pad="10"/>
+<wire x1="22.86" y1="-7.62" x2="63.5" y2="-121.92" width="0" layer="19" extent="1-1"/>
 </signal>
 <signal name="PA1">
 <contactref element="IC1" pad="39"/>
-<contactref element="PORTA" pad="2"/>
-<wire x1="22.86" y1="-10.16" x2="53.34" y2="-121.92" width="0" layer="19" extent="1-1"/>
+<contactref element="PORTA" pad="9"/>
+<wire x1="22.86" y1="-10.16" x2="63.5" y2="-124.46" width="0" layer="19" extent="1-1"/>
 </signal>
 <signal name="PA2">
 <contactref element="IC1" pad="38"/>
-<contactref element="PORTA" pad="3"/>
-<wire x1="22.86" y1="-12.7" x2="55.88" y2="-124.46" width="0" layer="19" extent="1-1"/>
+<contactref element="PORTA" pad="8"/>
+<wire x1="22.86" y1="-12.7" x2="60.96" y2="-121.92" width="0" layer="19" extent="1-1"/>
 </signal>
 <signal name="PA3">
 <contactref element="IC1" pad="37"/>
-<contactref element="PORTA" pad="4"/>
-<wire x1="22.86" y1="-15.24" x2="55.88" y2="-121.92" width="0" layer="19" extent="1-1"/>
+<contactref element="PORTA" pad="7"/>
+<wire x1="22.86" y1="-15.24" x2="60.96" y2="-124.46" width="0" layer="19" extent="1-1"/>
 </signal>
 <signal name="PA4">
 <contactref element="IC1" pad="36"/>
-<contactref element="PORTA" pad="5"/>
-<wire x1="22.86" y1="-17.78" x2="58.42" y2="-124.46" width="0" layer="19" extent="1-1"/>
+<contactref element="PORTA" pad="6"/>
+<wire x1="22.86" y1="-17.78" x2="58.42" y2="-121.92" width="0" layer="19" extent="1-1"/>
 </signal>
 <signal name="PA5">
 <contactref element="IC1" pad="35"/>
-<contactref element="PORTA" pad="6"/>
-<wire x1="22.86" y1="-20.32" x2="58.42" y2="-121.92" width="0" layer="19" extent="1-1"/>
+<contactref element="PORTA" pad="5"/>
+<wire x1="22.86" y1="-20.32" x2="58.42" y2="-124.46" width="0" layer="19" extent="1-1"/>
 </signal>
 <signal name="PA6">
 <contactref element="IC1" pad="34"/>
-<contactref element="PORTA" pad="7"/>
-<wire x1="22.86" y1="-22.86" x2="60.96" y2="-124.46" width="0" layer="19" extent="1-1"/>
+<contactref element="PORTA" pad="4"/>
+<wire x1="22.86" y1="-22.86" x2="55.88" y2="-121.92" width="0" layer="19" extent="1-1"/>
 </signal>
 <signal name="PA7">
 <contactref element="IC1" pad="33"/>
-<contactref element="PORTA" pad="8"/>
-<wire x1="22.86" y1="-25.4" x2="60.96" y2="-121.92" width="0" layer="19" extent="1-1"/>
+<contactref element="PORTA" pad="3"/>
+<wire x1="22.86" y1="-25.4" x2="55.88" y2="-124.46" width="0" layer="19" extent="1-1"/>
 </signal>
 <signal name="PC0">
 <contactref element="IC1" pad="22"/>
-<contactref element="PORTC" pad="1"/>
-<wire x1="22.86" y1="-53.34" x2="78.74" y2="-124.46" width="0" layer="19" extent="1-1"/>
+<contactref element="PORTC" pad="10"/>
+<wire x1="22.86" y1="-53.34" x2="88.9" y2="-121.92" width="0" layer="19" extent="1-1"/>
 </signal>
 <signal name="PC1">
 <contactref element="IC1" pad="23"/>
-<contactref element="PORTC" pad="2"/>
-<wire x1="22.86" y1="-50.8" x2="78.74" y2="-121.92" width="0" layer="19" extent="1-1"/>
+<contactref element="PORTC" pad="9"/>
+<wire x1="22.86" y1="-50.8" x2="88.9" y2="-124.46" width="0" layer="19" extent="1-1"/>
 </signal>
 <signal name="PC2">
 <contactref element="IC1" pad="24"/>
-<contactref element="PORTC" pad="3"/>
-<wire x1="22.86" y1="-48.26" x2="81.28" y2="-124.46" width="0" layer="19" extent="1-1"/>
+<contactref element="PORTC" pad="8"/>
+<wire x1="22.86" y1="-48.26" x2="86.36" y2="-121.92" width="0" layer="19" extent="1-1"/>
 </signal>
 <signal name="PC3">
 <contactref element="IC1" pad="25"/>
-<contactref element="PORTC" pad="4"/>
-<wire x1="22.86" y1="-45.72" x2="81.28" y2="-121.92" width="0" layer="19" extent="1-1"/>
+<contactref element="PORTC" pad="7"/>
+<wire x1="22.86" y1="-45.72" x2="86.36" y2="-124.46" width="0" layer="19" extent="1-1"/>
 </signal>
 <signal name="PC4">
 <contactref element="IC1" pad="26"/>
-<contactref element="PORTC" pad="5"/>
-<wire x1="22.86" y1="-43.18" x2="83.82" y2="-124.46" width="0" layer="19" extent="1-1"/>
+<contactref element="PORTC" pad="6"/>
+<wire x1="22.86" y1="-43.18" x2="83.82" y2="-121.92" width="0" layer="19" extent="1-1"/>
 </signal>
 <signal name="PC5">
 <contactref element="IC1" pad="27"/>
-<contactref element="PORTC" pad="6"/>
-<wire x1="22.86" y1="-40.64" x2="83.82" y2="-121.92" width="0" layer="19" extent="1-1"/>
+<contactref element="PORTC" pad="5"/>
+<wire x1="22.86" y1="-40.64" x2="83.82" y2="-124.46" width="0" layer="19" extent="1-1"/>
 </signal>
 <signal name="PC6">
 <contactref element="IC1" pad="28"/>
-<contactref element="PORTC" pad="7"/>
-<wire x1="22.86" y1="-38.1" x2="86.36" y2="-124.46" width="0" layer="19" extent="1-1"/>
+<contactref element="PORTC" pad="4"/>
+<wire x1="22.86" y1="-38.1" x2="81.28" y2="-121.92" width="0" layer="19" extent="1-1"/>
 </signal>
 <signal name="PC7">
 <contactref element="IC1" pad="29"/>
-<contactref element="PORTC" pad="8"/>
-<wire x1="22.86" y1="-35.56" x2="86.36" y2="-121.92" width="0" layer="19" extent="1-1"/>
+<contactref element="PORTC" pad="3"/>
+<wire x1="22.86" y1="-35.56" x2="81.28" y2="-124.46" width="0" layer="19" extent="1-1"/>
 </signal>
 <signal name="VIN_REG">
@@
 <contactref element="IC2" pad="3"/>
 <contactref element="IC1" pad="10"/>
-<contactref element="PORTA" pad="9"/>
-<contactref element="PORTC" pad="9"/>
 <contactref element="IC1" pad="30"/>
 <contactref element="C1" pad="1"/>
@@
 <contactref element="R3" pad="1"/>
 <contactref element="R4" pad="2"/>
+<contactref element="PORTC" pad="1"/>
+<contactref element="PORTA" pad="1"/>
 <wire x1="7.62" y1="-200.66" x2="15.24" y2="-245.11" width="0" layer="19" extent="1-1"/>
 <wire x1="15.24" y1="-186.69" x2="7.62" y2="-200.66" width="0" layer="19" extent="1-1"/>
@@
 <wire x1="29.21" y1="-143.51" x2="8.89" y2="-143.51" width="0" layer="19" extent="1-1"/>
 <wire x1="8.89" y1="-123.19" x2="8.89" y2="-143.51" width="0" layer="19" extent="1-1"/>
-<wire x1="63.5" y1="-124.46" x2="29.21" y2="-143.51" width="0" layer="19" extent="1-1"/>
-<wire x1="88.9" y1="-124.46" x2="63.5" y2="-124.46" width="0" layer="19" extent="1-1"/>
-<wire x1="67.31" y1="-158.75" x2="63.5" y2="-124.46" width="0" layer="19" extent="1-1"/>
+<wire x1="53.34" y1="-124.46" x2="29.21" y2="-143.51" width="0" layer="19" extent="1-1"/>
+<wire x1="78.74" y1="-124.46" x2="53.34" y2="-124.46" width="0" layer="19" extent="1-1"/>
+<wire x1="67.31" y1="-158.75" x2="78.74" y2="-124.46" width="0" layer="19" extent="1-1"/>
 <wire x1="22.86" y1="-33.02" x2="8.89" y2="-123.19" width="0" layer="19" extent="1-1"/>
 <wire x1="7.62" y1="-30.48" x2="22.86" y2="-33.02" width="0" layer="19" extent="1-1"/>
@@
 <wire x1="7.62" y1="-15.24" x2="7.62" y2="-214.63" width="0" layer="19" extent="1-1"/>
 </signal>
-<signal name="N$1">
-<contactref element="PORTC" pad="10"/>
-</signal>
-<signal name="N$2">
-<contactref element="PORTA" pad="10"/>
-</signal>
 <signal name="PB4">
 <contactref element="IC1" pad="5"/>
@@
 <wire x1="11.43" y1="-229.87" x2="7.62" y2="-245.11" width="0" layer="19" extent="1-1"/>
 </signal>
+<signal name="N$4">
+<contactref element="S1" pad="2"/>
+<contactref element="R3" pad="2"/>
+<wire x1="37.54" y1="-126.71" x2="15.24" y2="-200.66" width="0" layer="19" extent="1-1"/>
+</signal>
 </signals>

Commit message: add usb
Parts:
- added R5, R6: 68, rcl:0204/7
- added R7: 1.5K, rcl:0204/7
- added X1: (no value), con-cypressindustries:32005-601
- moved T3 230.0 mm to (213.4, -55.9), flipped to the bottom
- moved C1 227.8 mm to (212.1, -38.1), flipped to the bottom
- moved IC2 227.8 mm to (212.1, -68.6), flipped to the bottom
- moved LED5 227.8 mm to (212.1, -124.5), flipped to the bottom
- moved R4 225.5 mm to (210.8, -139.7), flipped to the bottom
- moved ICSP 225.5 mm to (210.8, -19.1), flipped to the bottom
- moved R1 225.5 mm to (210.8, -81.3), flipped to the bottom
- moved R2 225.5 mm to (210.8, -109.2), flipped to the bottom
- moved R3 225.5 mm to (210.8, -95.2), flipped to the bottom
- moved T4 197.0 mm to (194.3, -55.9), flipped to the bottom
- moved C2 192.7 mm to (191.8, -38.1), flipped to the bottom
- moved LED1 187.3 mm to (4.19, 39.4), flipped to the bottom, turned to 270 degrees
- moved S1 186.3 mm to (188.0, -19.1), flipped to the bottom
- moved LED2 180.7 mm to (4.19, 29.2), flipped to the bottom, turned to 270 degrees
- moved LED3 173.0 mm to (4.19, 16.5), flipped to the bottom, turned to 270 degrees
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Connections:
- removed net N$11: IC1.14
- removed net N$12: IC1.15
- new net N$1: X1.1
- new net N$2: R5.1, X1.3
- new net N$5: X1.4
- new net N$6: R6.1, R7.1, X1.2
- new net PD0: IC1.14, R2.1
- new net PD1: IC1.15, R1.1, U1.4
- net GND: now also X1.5
- net PB2: now also R5.2; no longer R1.1, U1.4
- net PB3: now also R6.2; no longer R2.1
- net VIN_REG: now also R7.2
Other:
- board size 100 x 80 mm -> 100 x 44.4 mm
