File: board files/v2.0/project_vostok_(tv_b_gone_extended)_v2.0.brd (EAGLE design)
At the start: 100 x 44 mm, 29 parts, among them IC1 ATMEGA644PV-10PU, IC2 MCP1825S-3302E_DB, Q5 MPS2907A, T1 2N3904, T2 2N3904, T3 2N3904, T4 2N3904, U1 PEC11R-4015F-S0024

Commit message: add version 2.0 files
Parts:
- moved S1 182.6 mm to (-68.6, 116.8), flipped to the top, turned to 0 degrees
- moved R6 171.5 mm to (-48.3, 128.3)
- moved XTL1 166.4 mm to (-66.0, 92.7), turned to 0 degrees
- moved X1 164.2 mm to (-54.6, 92.7), turned to 0 degrees
- moved LED5 159.3 mm to (-59.7, 118.1), turned to 0 degrees
- moved C2 158.5 mm to (-69.8, 108.0)
- moved R5 155.3 mm to (-38.1, 128.3)
- moved Q5 152.9 mm to (-78.7, 91.4), turned to 0 degrees
- moved R2 148.5 mm to (-78.7, 123.2)
- moved ICSP 146.1 mm to (-43.2, 95.2)
- moved PORTC 146.0 mm to (-53.3, 108.0), flipped to the top, turned to 0 degrees
- moved U1 142.2 mm to (-22.9, 96.5), flipped to the top, turned to 0 degrees
- moved T4 140.8 mm to (-61.0, 123.2), turned to 0 degrees
- moved C1 139.6 mm to (-63.5, 108.0)
- moved R1 138.6 mm to (-68.6, 123.2)
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Routing:
- net VIN_REG: track 200.7 -> 0.00 mm, vias 4 -> 0
- net VOUT_REG: track 159.1 -> 0.00 mm, vias 1 -> 0
- net PB3: track 92.7 -> 0.00 mm
- net Q5_E: track 92.4 -> 0.00 mm
- net PC1: track 87.4 -> 0.00 mm
- net PB2: track 85.7 -> 0.00 mm, vias 3 -> 0
- net MOSI: track 81.4 -> 0.00 mm, vias 3 -> 0
- net N$6: track 77.7 -> 0.00 mm, vias 2 -> 0
- net RESET: track 73.7 -> 0.00 mm, vias 2 -> 0
- net SCK: track 70.1 -> 0.00 mm, vias 2 -> 0
- net PD1: track 66.7 -> 0.00 mm, vias 1 -> 0
- net MISO: track 66.7 -> 0.00 mm, vias 2 -> 0
- net PA7: track 58.1 -> 0.00 mm
- net GND: track 54.7 -> 0.00 mm, vias 2 -> 0
- net XTAL1: track 51.5 -> 0.00 mm, vias 2 -> 0
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- removed copper zone on layer 16, net GND
Other:
- board size 100 x 44 mm -> 160 x 100 mm
- board text removed: "GND"
- board text removed: "MISO"
- board text removed: "MOSI"
- board text removed: "Project Vostok v1.1 Anton Nikitin - 2019"
- board text removed: "RST"
- board text removed: "SCK"
- board text removed: "VCC"
