File: board files/v2.0/project_vostok_(tv_b_gone_extended)_v2.0.sch (EAGLE design)
At the start: 29 parts, among them IC1 ATMEGA644PV-10PU, IC2 MCP1825S-3302E_DB, Q5 MPS2907A, T1 2N3904, T2 2N3904, T3 2N3904, T4 2N3904, U1 PEC11R-4015F-S0024, X1 MINI-USB_SHIELD5P2-32005-601

Commit message: add version 2.0 files
Other:
- note added: "v2.0"
- note removed: "v1.1"
Changed lines of the file:
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@@
 <text x="191.516" y="107.188" size="2.032" layer="94">Project Vostok - Anton Nikitin
 IR LED Circuit taken from TV-B-Gone</text>
-<text x="246.38" y="109.22" size="2.54" layer="94">v1.1</text>
+<text x="246.38" y="109.22" size="2.54" layer="94">v2.0</text>
 <text x="191.516" y="98.806" size="2.54" layer="94">CC 2.5 BY/SA</text>
 <wire x1="-86.36" y1="342.9" x2="0" y2="342.9" width="0.1524" layer="95" style="shortdash"/>
